Commit message: changed reward function + added diagnostic for nan

File: custom urdf/Tarot 650 Assembly_urdf_wts.SLDASM/urdf/Tarot 650 Assembly_urdf_wts.SLDASM.urdf (robot description, URDF)
Before this commit: robot Tarot 650 Assembly_urdf_wts.SLDASM, 5 links, 4 joints
Joints:
- joint Motor1: type continuous -> fixed
- joint Motor2: type continuous -> fixed
- joint Motor3: type continuous -> fixed
- joint Motor4: type continuous -> fixed
